File: nestDuinov5.kicad_pcb (KiCad board)
At the start: 2 copper layers, 68.6 x 53.3 mm, 34 parts, among them J1 Power, J2 Digital/PWM, J3 Analog, J4 Digital/PWM, J5 FTDI, J6 Barrel_Jack_Switch, J7 ISP, SW1 Reset, U1 AMS1117-3.3, U2 ATmega328P-P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

Commit message: Updated
Other:
- board text added: "https://github.com/ crnicholson/nestDuino"
- board text added: "nestDuino v6 Designed in MA, US, by Charles Nicholson, June 2024, for NESciTech."
- board text removed: "nestDuino v6 Designed in MA, US, by Charles Nicholson, June 2024, for NeSciTech."
Changed lines of the file:
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@@
 		(layer "Edge.Cuts")
 	)
-	(gr_text "nestDuino v6\nDesigned in MA, US, by Charles Nicholson, June 2024, for NeSciTech.\n"
+	(gr_text "nestDuino v6\nDesigned in MA, US, by Charles Nicholson, June 2024, for NESciTech.\n"
 		(at 163.5 53.391 0)
 		(layer "B.SilkS")
@@
 			)
 			(justify left bottom mirror)
+		)
+	)
+	(gr_text "https://github.com/\ncrnicholson/nestDuino"
+		(at 163.5 59.233 0)
+		(layer "B.SilkS")
+		(effects
+			(font
+				(size 1 1)
+				(thickness 0.15)
+			)
+			(justify left bottom mirror)

Commit message: Commit
Parts:
- C1, C10, C11, C12, C2, C3, C4, C5, C6, C7, C8: footprint Capacitor_THT:C_Disc_D4.3mm_W1.9mm_P5.00mm -> footprints:C_Disc_D4.3mm_W1.9mm_P5.00mm
- C9: footprint Capacitor_THT:CP_Radial_D5.0mm_P2.00mm -> footprints:CP_Radial_D5.0mm_P2.00mm
- D1, D2: footprint LED_THT:LED_D3.0mm -> footprints:LED_D3.0mm
- G***: footprint LOGO -> footprints:LOGO
- J1, J4: footprint Connector_PinSocket_2.54mm:PinSocket_1x08_P2.54mm_Vertical -> footprints:PinSocket_1x08_P2.54mm_Vertical
- J2: footprint Connector_PinSocket_2.54mm:PinSocket_1x10_P2.54mm_Vertical -> footprints:PinSocket_1x10_P2.54mm_Vertical
- J3: footprint Connector_PinSocket_2.54mm:PinSocket_1x06_P2.54mm_Vertical -> footprints:PinSocket_1x06_P2.54mm_Vertical
- J5: footprint Connector_PinSocket_2.54mm:PinSocket_1x06_P2.54mm_Horizontal -> footprints:PinSocket_1x06_P2.54mm_Horizontal
- J6: footprint Connector_BarrelJack:BarrelJack_Horizontal -> footprints:BarrelJack_Horizontal
- J7: footprint Connector_PinHeader_2.54mm:PinHeader_2x03_P2.54mm_Vertical -> footprints:PinHeader_2x03_P2.54mm_Vertical
- MH1, MH2, MH3, MH4: footprint Arduino_MountingHole:MountingHole_3.2mm -> footprints:MountingHole_3.2mm
- R1, R2, R3: footprint Resistor_THT:R_Axial_DIN0207_L6.3mm_D2.5mm_P10.16mm_Horizontal -> footprints:R_Axial_DIN0207_L6.3mm_D2.5mm_P10.16mm_Horizontal
- SW1: footprint Button_Switch_THT:SW_PUSH_6mm -> footprints:SW_PUSH_6mm
- U1: footprint Package_TO_SOT_SMD:SOT-223-3_TabPin2 -> footprints:SOT-223-3_TabPin2
- U2: footprint Package_DIP:DIP-28_W7.62mm -> footprints:DIP-28_W7.62mm
- U3: footprint Package_TO_SOT_THT:TO-220-3_Horizontal_TabDown -> footprints:TO-220-3_Horizontal_TabDown
- Y1: footprint Crystal:Crystal_HC49-U_Vertical -> footprints:Crystal_HC49-U_Vertical
